File: INA250A4.sch (KiCad schematic (older format))
At the start: 2 parts, among them U24 INA250A4PW

Commit message: Placement première charge active
Parts:
- renumbered C53 to C56, U24 to U27

Commit message: Debug routing
Changed lines of the file:
@@
 $Descr A4 11693 8268
 encoding utf-8
-Sheet 26 80
+Sheet 31 80
 Title ""
 Date "2020-05-19"
@@
 AR Path="/5EEC30AA/5EDDE040/5FCD7717" Ref="U20"  Part="1"
 AR Path="/5EEC30AA/5EDDE34E/5FCD7717" Ref="U21"  Part="1"
-F 0 "U27" H 5750 3537 60  0000 C CNN
+F 0 "U25" H 5750 3537 60  0000 C CNN
 F 1 "INA250A4PW" H 5750 3431 60  0000 C CNN
 F 2 "Package_SO:TSSOP-16_4.4x5mm_P0.65mm" H 5750 3390 60  0001 C CNN
@@
 AR Path="/5EEC30AA/5EDDE040/5EDB22E2" Ref="C49"  Part="1"
 AR Path="/5EEC30AA/5EDDE34E/5EDB22E2" Ref="C50"  Part="1"
-F 0 "C56" H 4315 4846 50  0000 L CNN
+F 0 "C54" H 4315 4846 50  0000 L CNN
 F 1 "0.1uF" H 4315 4755 50  0000 L CNN
 F 2 "Capacitor_SMD:C_0402_1005Metric" H 4238 4650 50  0001 C CNN
@@
 AR Path="/5EC4179E/5EDDE040/618429BE" Ref="#PWR0110"  Part="1"
 AR Path="/5EC4179E/5EDDE34E/618429BE" Ref="#PWR0113"  Part="1"
-F 0 "#PWR0116" H 6950 3700 50  0001 C CNN
+F 0 "#PWR0110" H 6950 3700 50  0001 C CNN
 F 1 "GNDA" H 6955 3777 50  0000 C CNN
 F 2 "" H 6950 3950 50  0001 C CNN
@@
 AR Path="/5EC4179E/5EDDE040/61842A2F" Ref="#PWR0108"  Part="1"
 AR Path="/5EC4179E/5EDDE34E/61842A2F" Ref="#PWR0111"  Part="1"
-F 0 "#PWR0114" H 3900 3700 50  0001 C CNN
+F 0 "#PWR0108" H 3900 3700 50  0001 C CNN
 F 1 "GNDA" H 3905 3777 50  0000 C CNN
 F 2 "" H 3900 3950 50  0001 C CNN
@@
 AR Path="/5EC4179E/5EDDE040/61842DA8" Ref="#PWR0109"  Part="1"
 AR Path="/5EC4179E/5EDDE34E/61842DA8" Ref="#PWR0112"  Part="1"
-F 0 "#PWR0115" H 4200 4900 50  0001 C CNN
+F 0 "#PWR0109" H 4200 4900 50  0001 C CNN
 F 1 "GNDA" H 4205 4977 50  0000 C CNN
 F 2 "" H 4200 5150 50  0001 C CNN

Commit message: retrait des test points inutiles
Changed lines of the file:
@@
 AR Path="/5EEC30AA/5EDDE040/5FCD7717" Ref="U20"  Part="1"
 AR Path="/5EEC30AA/5EDDE34E/5FCD7717" Ref="U21"  Part="1"
-F 0 "U25" H 5750 3537 60  0000 C CNN
+F 0 "U27" H 5750 3537 60  0000 C CNN
 F 1 "INA250A4PW" H 5750 3431 60  0000 C CNN
 F 2 "Package_SO:TSSOP-16_4.4x5mm_P0.65mm" H 5750 3390 60  0001 C CNN
@@
 AR Path="/5EEC30AA/5EDDE040/5EDB22E2" Ref="C49"  Part="1"
 AR Path="/5EEC30AA/5EDDE34E/5EDB22E2" Ref="C50"  Part="1"
-F 0 "C54" H 4315 4846 50  0000 L CNN
+F 0 "C56" H 4315 4846 50  0000 L CNN
 F 1 "0.1uF" H 4315 4755 50  0000 L CNN
 F 2 "Capacitor_SMD:C_0402_1005Metric" H 4238 4650 50  0001 C CNN
@@
 AR Path="/5EC4179E/5EDDE040/618429BE" Ref="#PWR0110"  Part="1"
 AR Path="/5EC4179E/5EDDE34E/618429BE" Ref="#PWR0113"  Part="1"
-F 0 "#PWR0110" H 6950 3700 50  0001 C CNN
+F 0 "#PWR0116" H 6950 3700 50  0001 C CNN
 F 1 "GNDA" H 6955 3777 50  0000 C CNN
 F 2 "" H 6950 3950 50  0001 C CNN
@@
 AR Path="/5EC4179E/5EDDE040/61842A2F" Ref="#PWR0108"  Part="1"
 AR Path="/5EC4179E/5EDDE34E/61842A2F" Ref="#PWR0111"  Part="1"
-F 0 "#PWR0108" H 3900 3700 50  0001 C CNN
+F 0 "#PWR0114" H 3900 3700 50  0001 C CNN
 F 1 "GNDA" H 3905 3777 50  0000 C CNN
 F 2 "" H 3900 3950 50  0001 C CNN
@@
 AR Path="/5EC4179E/5EDDE040/61842DA8" Ref="#PWR0109"  Part="1"
 AR Path="/5EC4179E/5EDDE34E/61842DA8" Ref="#PWR0112"  Part="1"
-F 0 "#PWR0109" H 4200 4900 50  0001 C CNN
+F 0 "#PWR0115" H 4200 4900 50  0001 C CNN
 F 1 "GNDA" H 4205 4977 50  0000 C CNN
 F 2 "" H 4200 5150 50  0001 C CNN

Commit message: routing usb
Changed lines of the file:
@@
 $Descr A4 11693 8268
 encoding utf-8
-Sheet 31 80
+Sheet 32 80
 Title ""
 Date "2020-05-19"
@@
 AR Path="/5EEC30AA/5EDDE040/5FCD7717" Ref="U20"  Part="1"
 AR Path="/5EEC30AA/5EDDE34E/5FCD7717" Ref="U21"  Part="1"
-F 0 "U27" H 5750 3537 60  0000 C CNN
+F 0 "U26" H 5750 3537 60  0000 C CNN
 F 1 "INA250A4PW" H 5750 3431 60  0000 C CNN
 F 2 "Package_SO:TSSOP-16_4.4x5mm_P0.65mm" H 5750 3390 60  0001 C CNN
@@
 AR Path="/5EEC30AA/5EDDE040/5EDB22E2" Ref="C49"  Part="1"
 AR Path="/5EEC30AA/5EDDE34E/5EDB22E2" Ref="C50"  Part="1"
-F 0 "C56" H 4315 4846 50  0000 L CNN
+F 0 "C55" H 4315 4846 50  0000 L CNN
 F 1 "0.1uF" H 4315 4755 50  0000 L CNN
 F 2 "Capacitor_SMD:C_0402_1005Metric" H 4238 4650 50  0001 C CNN
@@
 AR Path="/5EC4179E/5EDDE040/618429BE" Ref="#PWR0110"  Part="1"
 AR Path="/5EC4179E/5EDDE34E/618429BE" Ref="#PWR0113"  Part="1"
-F 0 "#PWR0116" H 6950 3700 50  0001 C CNN
+F 0 "#PWR0113" H 6950 3700 50  0001 C CNN
 F 1 "GNDA" H 6955 3777 50  0000 C CNN
 F 2 "" H 6950 3950 50  0001 C CNN
@@
 AR Path="/5EC4179E/5EDDE040/61842A2F" Ref="#PWR0108"  Part="1"
 AR Path="/5EC4179E/5EDDE34E/61842A2F" Ref="#PWR0111"  Part="1"
-F 0 "#PWR0114" H 3900 3700 50  0001 C CNN
+F 0 "#PWR0111" H 3900 3700 50  0001 C CNN
 F 1 "GNDA" H 3905 3777 50  0000 C CNN
 F 2 "" H 3900 3950 50  0001 C CNN
@@
 AR Path="/5EC4179E/5EDDE040/61842DA8" Ref="#PWR0109"  Part="1"
 AR Path="/5EC4179E/5EDDE34E/61842DA8" Ref="#PWR0112"  Part="1"
-F 0 "#PWR0115" H 4200 4900 50  0001 C CNN
+F 0 "#PWR0112" H 4200 4900 50  0001 C CNN
 F 1 "GNDA" H 4205 4977 50  0000 C CNN
 F 2 "" H 4200 5150 50  0001 C CNN

Commit message: Debut routing cannaux passifs
Changed lines of the file:
@@
 $Descr A4 11693 8268
 encoding utf-8
-Sheet 32 80
+Sheet 17 80
 Title ""
 Date "2020-05-19"
@@
 AR Path="/5EEC30AA/5EDDE040/5FCD7717" Ref="U20"  Part="1"
 AR Path="/5EEC30AA/5EDDE34E/5FCD7717" Ref="U21"  Part="1"
-F 0 "U26" H 5750 3537 60  0000 C CNN
+F 0 "U11" H 5750 3537 60  0000 C CNN
 F 1 "INA250A4PW" H 5750 3431 60  0000 C CNN
 F 2 "Package_SO:TSSOP-16_4.4x5mm_P0.65mm" H 5750 3390 60  0001 C CNN
@@
 AR Path="/5EEC30AA/5EDDE040/5EDB22E2" Ref="C49"  Part="1"
 AR Path="/5EEC30AA/5EDDE34E/5EDB22E2" Ref="C50"  Part="1"
-F 0 "C55" H 4315 4846 50  0000 L CNN
+F 0 "C40" H 4315 4846 50  0000 L CNN
 F 1 "0.1uF" H 4315 4755 50  0000 L CNN
 F 2 "Capacitor_SMD:C_0402_1005Metric" H 4238 4650 50  0001 C CNN
@@
 AR Path="/5EC4179E/5EDDE040/618429BE" Ref="#PWR0110"  Part="1"
 AR Path="/5EC4179E/5EDDE34E/618429BE" Ref="#PWR0113"  Part="1"
-F 0 "#PWR0113" H 6950 3700 50  0001 C CNN
+F 0 "#PWR071" H 6950 3700 50  0001 C CNN
 F 1 "GNDA" H 6955 3777 50  0000 C CNN
 F 2 "" H 6950 3950 50  0001 C CNN
@@
 AR Path="/5EC4179E/5EDDE040/61842A2F" Ref="#PWR0108"  Part="1"
 AR Path="/5EC4179E/5EDDE34E/61842A2F" Ref="#PWR0111"  Part="1"
-F 0 "#PWR0111" H 3900 3700 50  0001 C CNN
+F 0 "#PWR069" H 3900 3700 50  0001 C CNN
 F 1 "GNDA" H 3905 3777 50  0000 C CNN
 F 2 "" H 3900 3950 50  0001 C CNN
@@
 AR Path="/5EC4179E/5EDDE040/61842DA8" Ref="#PWR0109"  Part="1"
 AR Path="/5EC4179E/5EDDE34E/61842DA8" Ref="#PWR0112"  Part="1"
-F 0 "#PWR0112" H 4200 4900 50  0001 C CNN
+F 0 "#PWR070" H 4200 4900 50  0001 C CNN
 F 1 "GNDA" H 4205 4977 50  0000 C CNN
 F 2 "" H 4200 5150 50  0001 C CNN

Commit message: routing input canaux voltages
Changed lines of the file:
@@
 $Descr A4 11693 8268
 encoding utf-8
-Sheet 17 80
+Sheet 20 80
 Title ""
 Date "2020-05-19"
@@
 AR Path="/5EEC30AA/5EDDE040/5FCD7717" Ref="U20"  Part="1"
 AR Path="/5EEC30AA/5EDDE34E/5FCD7717" Ref="U21"  Part="1"
-F 0 "U11" H 5750 3537 60  0000 C CNN
+F 0 "U14" H 5750 3537 60  0000 C CNN
 F 1 "INA250A4PW" H 5750 3431 60  0000 C CNN
 F 2 "Package_SO:TSSOP-16_4.4x5mm_P0.65mm" H 5750 3390 60  0001 C CNN
@@
 AR Path="/5EEC30AA/5EDDE040/5EDB22E2" Ref="C49"  Part="1"
 AR Path="/5EEC30AA/5EDDE34E/5EDB22E2" Ref="C50"  Part="1"
-F 0 "C40" H 4315 4846 50  0000 L CNN
+F 0 "C43" H 4315 4846 50  0000 L CNN
 F 1 "0.1uF" H 4315 4755 50  0000 L CNN
 F 2 "Capacitor_SMD:C_0402_1005Metric" H 4238 4650 50  0001 C CNN
@@
 AR Path="/5EC4179E/5EDDE040/618429BE" Ref="#PWR0110"  Part="1"
 AR Path="/5EC4179E/5EDDE34E/618429BE" Ref="#PWR0113"  Part="1"
-F 0 "#PWR071" H 6950 3700 50  0001 C CNN
+F 0 "#PWR0116" H 6950 3700 50  0001 C CNN
 F 1 "GNDA" H 6955 3777 50  0000 C CNN
 F 2 "" H 6950 3950 50  0001 C CNN
@@
 AR Path="/5EC4179E/5EDDE040/61842A2F" Ref="#PWR0108"  Part="1"
 AR Path="/5EC4179E/5EDDE34E/61842A2F" Ref="#PWR0111"  Part="1"
-F 0 "#PWR069" H 3900 3700 50  0001 C CNN
+F 0 "#PWR0114" H 3900 3700 50  0001 C CNN
 F 1 "GNDA" H 3905 3777 50  0000 C CNN
 F 2 "" H 3900 3950 50  0001 C CNN
@@
 AR Path="/5EC4179E/5EDDE040/61842DA8" Ref="#PWR0109"  Part="1"
 AR Path="/5EC4179E/5EDDE34E/61842DA8" Ref="#PWR0112"  Part="1"
-F 0 "#PWR070" H 4200 4900 50  0001 C CNN
+F 0 "#PWR0115" H 4200 4900 50  0001 C CNN
 F 1 "GNDA" H 4205 4977 50  0000 C CNN
 F 2 "" H 4200 5150 50  0001 C CNN

Commit message: Changement pin pour switchs cannaux passifs
Changed lines of the file:
@@
 $Descr A4 11693 8268
 encoding utf-8
-Sheet 20 80
+Sheet 33 80
 Title ""
 Date "2020-05-19"
@@
 AR Path="/5EEC30AA/5EDDE040/5FCD7717" Ref="U20"  Part="1"
 AR Path="/5EEC30AA/5EDDE34E/5FCD7717" Ref="U21"  Part="1"
-F 0 "U14" H 5750 3537 60  0000 C CNN
+F 0 "U27" H 5750 3537 60  0000 C CNN
 F 1 "INA250A4PW" H 5750 3431 60  0000 C CNN
 F 2 "Package_SO:TSSOP-16_4.4x5mm_P0.65mm" H 5750 3390 60  0001 C CNN
@@
 AR Path="/5EEC30AA/5EDDE040/5EDB22E2" Ref="C49"  Part="1"
 AR Path="/5EEC30AA/5EDDE34E/5EDB22E2" Ref="C50"  Part="1"
-F 0 "C43" H 4315 4846 50  0000 L CNN
+F 0 "C56" H 4315 4846 50  0000 L CNN
 F 1 "0.1uF" H 4315 4755 50  0000 L CNN
 F 2 "Capacitor_SMD:C_0402_1005Metric" H 4238 4650 50  0001 C CNN
