File: temperature.sch (KiCad schematic (older format))
At the start: 20 parts, among them T1+1 TestPoint, T1-1 TestPoint, T2+1 TestPoint, T2-1 TestPoint, U4 ADS1118IDGS

Commit message: Placement première charge active
Changed lines of the file:
@@
 $Descr A4 11693 8268
 encoding utf-8
-Sheet 4 80
+Sheet 58 80
 Title "Acquisiton température"
 Date "2020-05-19"
@@
 AR Path="/5F466B56/5EB520F2" Ref="U34"  Part="1"
 AR Path="/5F466B61/5EB520F2" Ref="U35"  Part="1"
-F 0 "U6" H 7250 4400 50  0000 C CNN
+F 0 "U35" H 7250 4400 50  0000 C CNN
 F 1 "ADS1118IDGS" H 7250 4300 50  0000 C CNN
 F 2 "Package_SO:VSSOP-10_3x3mm_P0.5mm" H 6900 3750 50  0001 C CNN
@@
 AR Path="/5F466B56/5EC3D85A" Ref="C90"  Part="1"
 AR Path="/5F466B61/5EC3D85A" Ref="C97"  Part="1"
-F 0 "C28" H 5365 4896 50  0000 L CNN
+F 0 "C97" H 5365 4896 50  0000 L CNN
 F 1 "1uF" H 5365 4805 50  0000 L CNN
 F 2 "Capacitor_SMD:C_0402_1005Metric" H 5288 4700 50  0001 C CNN
@@
 AR Path="/5F466B56/5EC3D854" Ref="C88"  Part="1"
 AR Path="/5F466B61/5EC3D854" Ref="C95"  Part="1"
-F 0 "C26" H 5165 5346 50  0000 L CNN
+F 0 "C95" H 5165 5346 50  0000 L CNN
 F 1 "0.1uF" H 5165 5255 50  0000 L CNN
 F 2 "Capacitor_SMD:C_0402_1005Metric" H 5088 5150 50  0001 C CNN
@@
 AR Path="/5F466B56/5EC3D84E" Ref="C87"  Part="1"
 AR Path="/5F466B61/5EC3D84E" Ref="C94"  Part="1"
-F 0 "C25" H 4935 4354 50  0000 R CNN
+F 0 "C94" H 4935 4354 50  0000 R CNN
 F 1 "0.1uF" H 4935 4445 50  0000 R CNN
 F 2 "Capacitor_SMD:C_0402_1005Metric" H 5088 4250 50  0001 C CNN
@@
 AR Path="/5F466B56/5EC3D848" Ref="R116"  Part="1"
 AR Path="/5F466B61/5EC3D848" Ref="R124"  Part="1"
-F 0 "R28" V 4443 4650 50  0000 C CNN
+F 0 "R124" V 4443 4650 50  0000 C CNN
 F 1 "499" V 4534 4650 50  0000 C CNN
 F 2 "Resistor_SMD:R_0603_1608Metric" V 4580 4650 50  0001 C CNN
@@
 AR Path="/5F466B56/5EC3D842" Ref="R117"  Part="1"
 AR Path="/5F466B61/5EC3D842" Ref="R125"  Part="1"
-F 0 "R29" V 4443 5050 50  0000 C CNN
+F 0 "R125" V 4443 5050 50  0000 C CNN
 F 1 "499" V 4534 5050 50  0000 C CNN
 F 2 "Resistor_SMD:R_0603_1608Metric" V 4580 5050 50  0001 C CNN
@@
 AR Path="/5F466B56/5EC3D83C" Ref="R113"  Part="1"
 AR Path="/5F466B61/5EC3D83C" Ref="R121"  Part="1"
-F 0 "R25" H 4120 5346 50  0000 L CNN
+F 0 "R121" H 4120 5346 50  0000 L CNN
 F 1 "1M" H 4120 5255 50  0000 L CNN
 F 2 "Resistor_SMD:R_0805_2012Metric" V 3980 5300 50  0001 C CNN
@@
 AR Path="/5F466B56/5EC3D836" Ref="R112"  Part="1"
 AR Path="/5F466B61/5EC3D836" Ref="R120"  Part="1"
-F 0 "R24" H 4120 4446 50  0000 L CNN
+F 0 "R120" H 4120 4446 50  0000 L CNN
 F 1 "1M" H 4120 4355 50  0000 L CNN
 F 2 "Resistor_SMD:R_0805_2012Metric" V 3980 4400 50  0001 C CNN
@@
 AR Path="/5F466B56/5EBEC841" Ref="C91"  Part="1"
 AR Path="/5F466B61/5EBEC841" Ref="C98"  Part="1"
-F 0 "C29" H 6850 2950 50  0000 C CNN
+F 0 "C98" H 6850 2950 50  0000 C CNN
 F 1 "0.1uF" H 6850 3050 50  0000 C CNN
 F 2 "Capacitor_SMD:C_0402_1005Metric" H 6638 2850 50  0001 C CNN
@@
 AR Path="/5F466B56/5EC2636D" Ref="T2+7"  Part="1"
 AR Path="/5F466B61/5EC2636D" Ref="T2+8"  Part="1"
-F 0 "T2+3" H 4458 4368 50  0000 L CNN
+F 0 "T2+8" H 4458 4368 50  0000 L CNN
 F 1 "TestPoint" H 4458 4277 50  0000 L CNN
 F 2 "TestPoint:TestPoint_Pad_1.0x1.0mm" H 4600 4250 50  0001 C CNN
@@
 AR Path="/5F466B56/5EC467A6" Ref="T2-7"  Part="1"
 AR Path="/5F466B61/5EC467A6" Ref="T2-8"  Part="1"
-F 0 "T2-3" H 4050 5600 50  0000 L CNN
+F 0 "T2-8" H 4050 5600 50  0000 L CNN
 F 1 "TestPoint" H 4000 5500 50  0000 L CNN
 F 2 "TestPoint:TestPoint_Pad_1.0x1.0mm" H 4600 5450 50  0001 C CNN
@@
 AR Path="/5F466B56/5EC22011" Ref="T1-7"  Part="1"
 AR Path="/5F466B61/5EC22011" Ref="T1-8"  Part="1"
-F 0 "T1-3" H 4050 3500 50  0000 L CNN
+F 0 "T1-8" H 4050 3500 50  0000 L CNN
 F 1 "TestPoint" H 4000 3400 50  0000 L CNN
 F 2 "TestPoint:TestPoint_Pad_1.0x1.0mm" H 4600 3350 50  0001 C CNN
@@
 AR Path="/5F466B56/5EC1E92D" Ref="T1+7"  Part="1"
 AR Path="/5F466B61/5EC1E92D" Ref="T1+8"  Part="1"
-F 0 "T1+3" H 4458 2268 50  0000 L CNN
+F 0 "T1+8" H 4458 2268 50  0000 L CNN
 F 1 "TestPoint" H 4458 2177 50  0000 L CNN
 F 2 "TestPoint:TestPoint_Pad_1.0x1.0mm" H 4600 2150 50  0001 C CNN
@@
 AR Path="/5F466B56/5EC09C7B" Ref="R110"  Part="1"
 AR Path="/5F466B61/5EC09C7B" Ref="R118"  Part="1"
-F 0 "R22" H 4120 2346 50  0000 L CNN
+F 0 "R118" H 4120 2346 50  0000 L CNN
 F 1 "1M" H 4120 2255 50  0000 L CNN
 F 2 "Resistor_SMD:R_0805_2012Metric" V 3980 2300 50  0001 C CNN
@@
 AR Path="/5F466B56/5EC0F883" Ref="R111"  Part="1"
 AR Path="/5F466B61/5EC0F883" Ref="R119"  Part="1"
-F 0 "R23" H 4120 3246 50  0000 L CNN
+F 0 "R119" H 4120 3246 50  0000 L CNN
 F 1 "1M" H 4120 3155 50  0000 L CNN
 F 2 "Resistor_SMD:R_0805_2012Metric" V 3980 3200 50  0001 C CNN
@@
 AR Path="/5F466B56/5EC11D48" Ref="R115"  Part="1"
 AR Path="/5F466B61/5EC11D48" Ref="R123"  Part="1"
-F 0 "R27" V 4443 2950 50  0000 C CNN
+F 0 "R123" V 4443 2950 50  0000 C CNN
 F 1 "499" V 4534 2950 50  0000 C CNN
 F 2 "Resistor_SMD:R_0603_1608Metric" V 4580 2950 50  0001 C CNN
@@
 AR Path="/5F466B56/5EC12ACC" Ref="R114"  Part="1"
 AR Path="/5F466B61/5EC12ACC" Ref="R122"  Part="1"
-F 0 "R26" V 4443 2550 50  0000 C CNN
+F 0 "R122" V 4443 2550 50  0000 C CNN
 F 1 "499" V 4534 2550 50  0000 C CNN
 F 2 "Resistor_SMD:R_0603_1608Metric" V 4580 2550 50  0001 C CNN
@@
 AR Path="/5F466B56/5EC13396" Ref="C85"  Part="1"
 AR Path="/5F466B61/5EC13396" Ref="C92"  Part="1"
-F 0 "C23" H 4935 2254 50  0000 R CNN
+F 0 "C92" H 4935 2254 50  0000 R CNN
 F 1 "0.1uF" H 4935 2345 50  0000 R CNN
 F 2 "Capacitor_SMD:C_0402_1005Metric" H 5088 2150 50  0001 C CNN
@@
 AR Path="/5F466B56/5EC146F1" Ref="C86"  Part="1"
 AR Path="/5F466B61/5EC146F1" Ref="C93"  Part="1"
-F 0 "C24" H 5165 3246 50  0000 L CNN
+F 0 "C93" H 5165 3246 50  0000 L CNN
 F 1 "0.1uF" H 5165 3155 50  0000 L CNN
 F 2 "Capacitor_SMD:C_0402_1005Metric" H 5088 3050 50  0001 C CNN
@@
 AR Path="/5F466B56/5EC15202" Ref="C89"  Part="1"
 AR Path="/5F466B61/5EC15202" Ref="C96"  Part="1"
-F 0 "C27" H 5365 2796 50  0000 L CNN
+F 0 "C96" H 5365 2796 50  0000 L CNN
 F 1 "1uF" H 5365 2705 50  0000 L CNN
 F 2 "Capacitor_SMD:C_0402_1005Metric" H 5288 2600 50  0001 C CNN
@@
 AR Path="/5F466B56/618455B5" Ref="#PWR0188"  Part="1"
 AR Path="/5F466B61/618455B5" Ref="#PWR0196"  Part="1"
-F 0 "#PWR044" H 6950 4200 50  0001 C CNN
+F 0 "#PWR0196" H 6950 4200 50  0001 C CNN
 F 1 "GNDA" H 6955 4277 50  0000 C CNN
 F 2 "" H 6950 4450 50  0001 C CNN
@@
 AR Path="/5F466B56/61845768" Ref="#PWR0187"  Part="1"
 AR Path="/5F466B61/61845768" Ref="#PWR0195"  Part="1"
-F 0 "#PWR043" H 6600 2900 50  0001 C CNN
+F 0 "#PWR0195" H 6600 2900 50  0001 C CNN
 F 1 "GNDA" H 6605 2977 50  0000 C CNN
 F 2 "" H 6600 3150 50  0001 C CNN
@@
 AR Path="/5F466B56/61845B4A" Ref="#PWR0186"  Part="1"
 AR Path="/5F466B61/61845B4A" Ref="#PWR0194"  Part="1"
-F 0 "#PWR042" H 5050 5200 50  0001 C CNN
+F 0 "#PWR0194" H 5050 5200 50  0001 C CNN
 F 1 "GNDA" H 5055 5277 50  0000 C CNN
 F 2 "" H 5050 5450 50  0001 C CNN
@@
 AR Path="/5F466B56/61846A90" Ref="#PWR0182"  Part="1"
 AR Path="/5F466B61/61846A90" Ref="#PWR0190"  Part="1"
-F 0 "#PWR038" H 4050 5200 50  0001 C CNN
+F 0 "#PWR0190" H 4050 5200 50  0001 C CNN
 F 1 "GNDA" H 4055 5277 50  0000 C CNN
 F 2 "" H 4050 5450 50  0001 C CNN
@@
 AR Path="/5F466B56/61846F48" Ref="#PWR0184"  Part="1"
 AR Path="/5F466B61/61846F48" Ref="#PWR0192"  Part="1"
-F 0 "#PWR040" H 5050 3100 50  0001 C CNN
+F 0 "#PWR0192" H 5050 3100 50  0001 C CNN
 F 1 "GNDA" H 5055 3177 50  0000 C CNN
 F 2 "" H 5050 3350 50  0001 C CNN
@@
 AR Path="/5F466B56/618474E2" Ref="#PWR0181"  Part="1"
 AR Path="/5F466B61/618474E2" Ref="#PWR0189"  Part="1"
-F 0 "#PWR037" H 4050 3100 50  0001 C CNN
+F 0 "#PWR0189" H 4050 3100 50  0001 C CNN
 F 1 "GNDA" H 4055 3177 50  0000 C CNN
 F 2 "" H 4050 3350 50  0001 C CNN
@@
 AR Path="/5F466B56/6184779B" Ref="#PWR0185"  Part="1"
 AR Path="/5F466B61/6184779B" Ref="#PWR0193"  Part="1"
-F 0 "#PWR041" H 5050 4000 50  0001 C CNN
+F 0 "#PWR0193" H 5050 4000 50  0001 C CNN
 F 1 "GNDA" H 5055 4077 50  0000 C CNN
 F 2 "" H 5050 4250 50  0001 C CNN
@@
 AR Path="/5F466B56/6184B7DC" Ref="#PWR0183"  Part="1"
 AR Path="/5F466B61/6184B7DC" Ref="#PWR0191"  Part="1"
-F 0 "#PWR039" H 5050 1900 50  0001 C CNN
+F 0 "#PWR0191" H 5050 1900 50  0001 C CNN
 F 1 "GNDA" H 5055 1977 50  0000 C CNN
 F 2 "" H 5050 2150 50  0001 C CNN
