File: PCB.kicad_pcb (KiCad board)
At the start: 4 copper layers, 200 x 150 mm, 517 parts, among them J1 PASSIVE_CHANNELS, J10 USB_RASPBERRY, J11 USB_ARDUINO, J12 100W_ch+, J13 100W_ch-, J14 100W_sense, J15 PowerMosGate, J16 PowerMosDrain, J2 PASSIVE_CHANNELS, J3 PASSIVE_CHANNELS, J4 12V+, J5 12V-, J6 5V_PI, J7 5V_PI, J8 ACTIVE_5W_CHANNELS, J9 5V_PI, Q1 BT137-600, Q10 IRLB3813PBF, Q11 IRLB3813PBF, Q12 IRLB3813PbF, Q13 IRLB3813PbF, Q14 IRLB3813PbF, Q15 IRLB3813PbF, Q16 IRLB3813PbF, Q17 IRLB3813PbF, Q2 IRLB3813PbF, Q3 IRLB3813PbF, Q4 IRLB3813PBF, Q5 IRLB3813PBF, Q6 IRLB3813PBF, Q7 IRLB3813PBF, Q8 IRLB3813PBF, Q9 IRLB3813PBF, SW1 RESET_SW, T1+1 TestPoint, T1+2 TestPoint, T1+3 TestPoint, T1+4 TestPoint, T1+5 TestPoint, T1+6 TestPoint, T1+7 TestPoint, T1+8 TestPoint, T1-1 TestPoint, T1-2 TestPoint, T1-3 TestPoint, T1-4 TestPoint, T1-5 TestPoint, T1-6 TestPoint, T1-7 TestPoint, T1-8 TestPoint, T2+1 TestPoint, T2+2 TestPoint, T2+3 TestPoint, T2+4 TestPoint, T2+5 TestPoint, T2+6 TestPoint, T2+7 TestPoint, T2+8 TestPoint, T2-1 TestPoint, T2-2 TestPoint, T2-3 TestPoint, T2-4 TestPoint, T2-5 TestPoint, T2-6 TestPoint, T2-7 TestPoint, T2-8 TestPoint, U1 LM431ACM3_NOPB, U10 INA250A4PW, U11 INA250A4PW, U12 INA250A4PW, U13 ADC124S021CIMM_NOPB, U14 INA250A4PW, U15 INA250A4PW, U16 INA250A4PW, U17 INA250A4PW, U18 ADC124S021CIMM_NOPB, U19 INA250A4PW, U2 LM1117-ADJ, U20 INA250A4PW, U21 INA250A4PW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

Commit message: Debug routing
Parts:
- moved F2 20.9 mm to (139.1, 188.6)
- moved F3 17.9 mm to (160.5, 188.6)
- moved J6 15.0 mm to (133.0, 203.0)
Routing:
- net /T1-: track 0.00 -> 8.24 mm
- net Net-(C16-Pad1): track 0.00 -> 8.08 mm
- net /T1+: track 0.00 -> 7.79 mm
- net Net-(C13-Pad1): track 0.00 -> 7.57 mm
- net Net-(C12-Pad1): track 0.00 -> 7.47 mm
- net Net-(C19-Pad1): track 0.00 -> 7.11 mm
- net Net-(C10-Pad1): track 0.00 -> 6.72 mm
- net Net-(C17-Pad1): track 0.00 -> 6.53 mm
- net Net-(C11-Pad1): track 0.00 -> 5.90 mm
- net Net-(C18-Pad1): track 0.00 -> 5.90 mm
Changed lines of the file:
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@@
     (thickness 1.6)
     (drawings 5)
-    (tracks 2)
+    (tracks 58)
     (zones 0)
     (modules 517)
@@
     (1 In1_Vert.Cu signal hide)
     (2 In2_Hor.Cu signal hide)
-    (31 B.Cu power)
+    (31 B.Cu power hide)
     (34 B.Paste user)
     (35 F.Paste user)
@@
     (44 Edge.Cuts user)
     (45 Margin user)
-    (46 B.CrtYd user hide)
+    (46 B.CrtYd user)
     (47 F.CrtYd user hide)
     (48 B.Fab user)
@@
     (tags capacitor)
     (attr smd)
-    (fp_text reference C9 (at -0.2 1.2) (layer F.SilkS)
+    (fp_text reference C9 (at -0.064 1.15) (layer F.SilkS)
       (effects (font (size 1 1) (thickness 0.15)))
     )
@@
     (tags capacitor)
     (attr smd)
-    (fp_text reference C11 (at 0 1) (layer F.SilkS)
+    (fp_text reference C11 (at 0 1.2) (layer F.SilkS)
       (effects (font (size 1 1) (thickness 0.15)))
     )
@@
     (tags capacitor)
     (attr smd)
-    (fp_text reference C12 (at -0.025 -0.9) (layer F.SilkS)
+    (fp_text reference C12 (at 0 -1.17) (layer F.SilkS)
       (effects (font (size 1 1) (thickness 0.15)))
     )
@@
   )
   (module PCB:Fuse5x15mm (layer F.Cu)
-    (at 160 188)
+    (at 139.1 188.6)
     (fp_text reference F2 (at 0 -4) (layer F.SilkS)
       (effects (font (size 1 1) (thickness 0.15)))
@@
   )
   (module PCB:Fuse5x15mm (layer F.Cu)
-    (at 160 170.75)
+    (at 160.5 188.6)
     (fp_text reference F3 (at 0 -4) (layer F.SilkS)
       (effects (font (size 1 1) (thickness 0.15)))
@@
   )
   (module TerminalBlock_Phoenix:TerminalBlock_Phoenix_PT-1,5-2-5.0-H_1x02_P5.00mm_Horizontal (layer F.Cu)
-    (at 133 188 270)
+    (at 133 203 270)
     (descr "Terminal Block Phoenix PT-1,5-2-5.0-H, 2 pins, pitch 5mm, size 10x9mm^2, drill diamater 1.3mm, pad diameter 2.6mm, see http://www.mouser.com/ds/2/324/ItemDetail_1935161-922578.pdf, script-generated using https://github.com/pointhi/kicad-footprint-generator/scripts/TerminalBlock_Phoenix")
     (tags "THT Terminal Block Phoenix PT-1,5-2-5.0-H pitch 5mm size 10x9mm^2 drill 1.3mm pad 2.6mm")
@@
       (effects (font (size 1 1) (thickness 0.15)))
     )
-    (fp_text user %R (at 0 0 270) (layer F.Fab)
+    (fp_text user %R (at 0.004 -0.038 270) (layer F.Fab)
       (effects (font (size 0.5 0.5) (thickness 0.08)))
     )
@@
   (gr_line (start 126 72) (end 326 72) (layer Edge.Cuts) (width 0.1))
   (gr_line (start 126 222) (end 126 72) (layer Edge.Cuts) (width 0.1))
+  (segment (start 142.765 198.426) (end 143.991 197.2) (width 0.2) (layer F.Cu) (net 7))
+  (segment (start 142.765 198.746) (end 142.765 198.426) (width 0.2) (layer F.Cu) (net 7))
+  (segment (start 143.991 197.2) (end 145.7 197.2) (width 0.2) (layer F.Cu) (net 7))
+  (segment (start 142.2 202.3585) (end 142.2 201) (width 0.2) (layer F.Cu) (net 7))
+  (segment (start 142.2 201) (end 142.2 199.4) (width 0.2) (layer F.Cu) (net 7))
+  (segment (start 142.2 199.4) (end 142.8 198.8) (width 0.2) (layer F.Cu) (net 7))
+  (segment (start 146.4 197.7) (end 146.25 197.85) (width 0.2) (layer F.Cu) (net 8))
+  (segment (start 143.735 199.066) (end 144.5 199.831) (width 0.2) (layer F.Cu) (net 8))
+  (segment (start 143.735 198.746) (end 143.735 199.066) (width 0.2) (layer F.Cu) (net 8))
+  (segment (start 144.5 199.831) (end 144.5 199.967876) (width 0.2) (layer F.Cu) (net 8))
+  (segment (start 144.5 199.967876) (end 144.5 202.25) (width 0.2) (layer F.Cu) (net 8))
+  (segment (start 143.735 198.426) (end 144.461 197.7) (width 0.2) (layer F.Cu) (net 8))
+  (segment (start 143.735 198.746) (end 143.735 198.426) (width 0.2) (layer F.Cu) (net 8))
+  (segment (start 144.461 197.7) (end 145.8 197.7) (width 0.2) (layer F.Cu) (net 8))
+  (segment (start 152 202.3585) (end 152 201) (width 0.2) (layer F.Cu) (net 9))
+  (segment (start 152 201) (end 152 199.5) (width 0.2) (layer F.Cu) (net 9))
+  (segment (start 152 199.5) (end 152.75 198.75) (width 0.2) (layer F.Cu) (net 9))
+  (segment (start 152.765 198.426) (end 152.039 197.7) (width 0.2) (layer F.Cu) (net 9))
+  (segment (start 152.765 198.746) (end 152.765 198.426) (width 0.2) (layer F.Cu) (net 9))
+  (segment (start 152.039 197.7) (end 151.4 197.7) (width 0.2) (layer F.Cu) (net 9))
+  (segment (start 154.6 202.271) (end 154.6 201.1) (width 0.2) (layer F.Cu) (net 10))
+  (segment (start 154.6 201.1) (end 154.6 199.6) (width 0.2) (layer F.Cu) (net 10))
+  (segment (start 154.6 199.6) (end 153.8 198.8) (width 0.2) (layer F.Cu) (net 10))
+  (segment (start 151.6 197.2) (end 150.9 197.2) (width 0.2) (layer F.Cu) (net 10))
+  (segment (start 152.509 197.2) (end 151.6 197.2) (width 0.2) (layer F.Cu) (net 10))
+  (segment (start 153.735 198.426) (end 152.509 197.2) (width 0.2) (layer F.Cu) (net 10))
+  (segment (start 153.735 198.746) (end 153.735 198.426) (width 0.2) (layer F.Cu) (net 10))
+  (segment (start 162.2 202.3585) (end 162.2 201.921) (width 0.2) (layer F.Cu) (net 12))
+  (segment (start 162.2 202.3585) (end 162.2 199.328124) (width 0.2) (layer F.Cu) (net 12))
+  (segment (start 163.991 197.2) (end 165.8 197.2) (width 0.2) (layer F.Cu) (net 12))
+  (segment (start 162.765 198.746) (end 162.765 198.426) (width 0.2) (layer F.Cu) (net 12))
+  (segment (start 162.765 198.426) (end 163.991 197.2) (width 0.2) (layer F.Cu) (net 12))
+  (segment (start 162.2 199.328124) (end 162.728124 198.8) (width 0.2) (layer F.Cu) (net 12))
+  (segment (start 163.735 198.426) (end 164.461 197.7) (width 0.2) (layer F.Cu) (net 13))
+  (segment (start 163.735 198.746) (end 163.735 198.426) (width 0.2) (layer F.Cu) (net 13))
+  (segment (start 164.461 197.7) (end 165.8 197.7) (width 0.2) (layer F.Cu) (net 13))
+  (segment (start 164.5 202.3585) (end 164.5 201.921) (width 0.2) (layer F.Cu) (net 13))
+  (segment (start 164.5 201.921) (end 164.5 199.5) (width 0.2) (layer F.Cu) (net 13))
+  (segment (start 164.5 199.5) (end 163.8 198.8) (width 0.2) (layer F.Cu) (net 13))
+  (segment (start 172 202.3585) (end 172 201.921) (width 0.2) (layer F.Cu) (net 14))
+  (segment (start 172 201.921) (end 172 199.5) (width 0.2) (layer F.Cu) (net 14))
+  (segment (start 172 199.5) (end 172.8 198.7) (width 0.2) (layer F.Cu) (net 14))
+  (segment (start 172.8 198.7) (end 171.8 197.7) (width 0.2) (layer F.Cu) (net 14))
+  (segment (start 171.8 197.7) (end 171.3 197.7) (width 0.2) (layer F.Cu) (net 14))
+  (segment (start 174.6 202.271) (end 174.6 201.8335) (width 0.2) (layer F.Cu) (net 15))
+  (segment (start 174.6 201.8335) (end 174.6 199.6) (width 0.2) (layer F.Cu) (net 15))
+  (segment (start 174.6 199.6) (end 173.7 198.7) (width 0.2) (layer F.Cu) (net 15))
+  (segment (start 173.735 198.426) (end 172.509 197.2) (width 0.2) (layer F.Cu) (net 15))
+  (segment (start 173.735 198.746) (end 173.735 198.426) (width 0.2) (layer F.Cu) (net 15))
+  (segment (start 172.509 197.2) (end 171.4 197.2) (width 0.2) (layer F.Cu) (net 15))
   (segment (start 314 139) (end 314 140.838477) (width 0.2) (layer B.Cu) (net 82))
+  (segment (start 141 209.5) (end 141 205.25) (width 0.2) (layer F.Cu) (net 102))
+  (segment (start 141 205.25) (end 142.25 204) (width 0.2) (layer F.Cu) (net 102))
+  (segment (start 141 205.25) (end 139.75 204) (width 0.2) (layer F.Cu) (net 102))
+  (segment (start 146 209.5) (end 146 205.5) (width 0.2) (layer F.Cu) (net 103))
+  (segment (start 146 205.5) (end 144.5 204) (width 0.2) (layer F.Cu) (net 103))
+  (segment (start 146 205.5) (end 147.5 204) (width 0.2) (layer F.Cu) (net 103))
   (segment (start 202.4286 181.487) (end 202.454 181.487) (width 0.2) (layer F.Cu) (net 190))
   (zone (net 2) (net_name GND) (layer B.Cu) (hatch edge 0.508)

Commit message: Routing initial température
Parts:
- moved SW1 9.76 mm to (201.6, 129.0)
- moved C15 1.31 mm to (148.7, 194.3)
- moved C22 1.31 mm to (168.7, 194.3)
- moved C29 1.31 mm to (188.7, 194.3)
- moved C36 1.31 mm to (208.7, 194.3)
Routing:
- net /MOSI: track 0.00 -> 70.1 mm, vias 0 -> 4
- net /MISO: track 0.00 -> 70.0 mm, vias 0 -> 4
- net /+5V: track 0.00 -> 47.7 mm
- net /T2+: track 0.00 -> 7.99 mm
- net /T2-: track 0.00 -> 7.68 mm
- net Net-(C23-Pad1): track 0.00 -> 7.61 mm
- net Net-(C30-Pad1): track 0.00 -> 7.56 mm
- net Net-(C26-Pad1): track 0.00 -> 6.85 mm
- net Net-(C33-Pad1): track 0.00 -> 6.80 mm
- net Net-(C31-Pad1): track 0.00 -> 6.40 mm
- net Net-(C24-Pad1): track 0.00 -> 6.40 mm
- net Net-(C32-Pad1): track 0.00 -> 5.82 mm
- net Net-(C25-Pad1): track 0.00 -> 5.75 mm
- net /SCK: track 0.00 -> 2.46 mm, vias 0 -> 1
