File: ChanelProtection.sch (KiCad schematic (older format))
At the start: 2 parts

Commit message: Placement canal passif intial
Changed lines of the file:
@@
 AR Path="/5F1340AA/5FCD1E19" Ref="#PWR0268"  Part="1"
 AR Path="/5F5525AA/5FCD1E19" Ref="#PWR0269"  Part="1"
-F 0 "#PWR0269" H 3250 3900 50  0001 C CNN
+F 0 "#PWR0207" H 3250 3900 50  0001 C CNN
 F 1 "GNDA" H 3255 3977 50  0000 C CNN
 F 2 "" H 3250 4150 50  0001 C CNN
@@
 AR Path="/5F1340AA/5FCD4D15" Ref="D18"  Part="1"
 AR Path="/5F5525AA/5FCD4D15" Ref="D19"  Part="1"
-F 0 "D19" V 3204 3879 50  0000 L CNN
+F 0 "D2" V 3204 3879 50  0000 L CNN
 F 1 "SMAJ9.0CA-E3/61" V 3295 3879 50  0000 L CNN
 F 2 "Diode_SMD:D_SMA" H 3250 3800 50  0001 C CNN
@@
 AR Path="/5F1340AA/5FCD5B9E" Ref="L18"  Part="1"
 AR Path="/5F5525AA/5FCD5B9E" Ref="L19"  Part="1"
-F 0 "L19" V 3619 3350 50  0000 C CNN
+F 0 "L2" V 3619 3350 50  0000 C CNN
 F 1 "L" V 3710 3350 50  0000 C CNN
 F 2 "PCB:TraceInductor" H 3800 3350 50  0001 C CNN

Commit message: Placement première charge active
Changed lines of the file:
@@
 $Descr A4 11693 8268
 encoding utf-8
-Sheet 60 80
+Sheet 77 80
 Title ""
 Date ""
@@
 AR Path="/5F1340AA/5FCD1E19" Ref="#PWR0268"  Part="1"
 AR Path="/5F5525AA/5FCD1E19" Ref="#PWR0269"  Part="1"
-F 0 "#PWR0207" H 3250 3900 50  0001 C CNN
+F 0 "#PWR0269" H 3250 3900 50  0001 C CNN
 F 1 "GNDA" H 3255 3977 50  0000 C CNN
 F 2 "" H 3250 4150 50  0001 C CNN
@@
 AR Path="/5F1340AA/5FCD4D15" Ref="D18"  Part="1"
 AR Path="/5F5525AA/5FCD4D15" Ref="D19"  Part="1"
-F 0 "D2" V 3204 3879 50  0000 L CNN
+F 0 "D19" V 3204 3879 50  0000 L CNN
 F 1 "SMAJ9.0CA-E3/61" V 3295 3879 50  0000 L CNN
 F 2 "Diode_SMD:D_SMA" H 3250 3800 50  0001 C CNN
@@
 AR Path="/5F1340AA/5FCD5B9E" Ref="L18"  Part="1"
 AR Path="/5F5525AA/5FCD5B9E" Ref="L19"  Part="1"
-F 0 "L2" V 3619 3350 50  0000 C CNN
+F 0 "L19" V 3619 3350 50  0000 C CNN
 F 1 "L" V 3710 3350 50  0000 C CNN
 F 2 "PCB:TraceInductor" H 3800 3350 50  0001 C CNN

Commit message: routing usb
Changed lines of the file:
@@
 $Descr A4 11693 8268
 encoding utf-8
-Sheet 80 80
+Sheet 67 80
 Title ""
 Date ""
@@
 AR Path="/5F1340AA/5FCD1E19" Ref="#PWR0267"  Part="1"
 AR Path="/5F5525AA/5FCD1E19" Ref="#PWR0268"  Part="1"
-F 0 "#PWR0268" H 3250 3900 50  0001 C CNN
+F 0 "#PWR0213" H 3250 3900 50  0001 C CNN
 F 1 "GNDA" H 3255 3977 50  0000 C CNN
 F 2 "" H 3250 4150 50  0001 C CNN
@@
 AR Path="/5F1340AA/5FCD4D15" Ref="D18"  Part="1"
 AR Path="/5F5525AA/5FCD4D15" Ref="D19"  Part="1"
-F 0 "D19" V 3204 3879 50  0000 L CNN
+F 0 "D9" V 3204 3879 50  0000 L CNN
 F 1 "SMAJ9.0CA-E3/61" V 3295 3879 50  0000 L CNN
 F 2 "Diode_SMD:D_SMA" H 3250 3800 50  0001 C CNN
@@
 AR Path="/5F1340AA/5FCD5B9E" Ref="L18"  Part="1"
 AR Path="/5F5525AA/5FCD5B9E" Ref="L19"  Part="1"
-F 0 "L19" V 3619 3350 50  0000 C CNN
+F 0 "L9" V 3619 3350 50  0000 C CNN
 F 1 "L" V 3710 3350 50  0000 C CNN
 F 2 "PCB:TraceInductor" H 3800 3350 50  0001 C CNN
