File: ChargeActive100W.sch (KiCad schematic (older format))
At the start: 26 parts, among them J15 PowerMosGate, J16 PowerMosDrain, J17 PowerMosSource, U36 LM358

Commit message: Placement première charge active
Parts:
- renumbered TPV+3 to TPV+1, TPV-3 to TPV-1, TPVAD3 to TPVAD1
Changed lines of the file:
@@
 Connection ~ 4850 3750
 $Comp
-L Connector:TestPoint TPV-3
+L Connector:TestPoint TPV-1
 U 1 1 5EF281AD
 P 4100 4000
-F 0 "TPV-3" H 4158 4118 50  0000 L CNN
+F 0 "TPV-1" H 4158 4118 50  0000 L CNN
 F 1 "TestPoint" H 4158 4027 50  0000 L CNN
 F 2 "TestPoint:TestPoint_Pad_1.0x1.0mm" H 4300 4000 50  0001 C CNN
@@
 $EndComp
 $Comp
-L Connector:TestPoint TPV+3
+L Connector:TestPoint TPV+1
 U 1 1 5EF2916C
 P 5200 3350
-F 0 "TPV+3" H 5258 3468 50  0000 L CNN
+F 0 "TPV+1" H 5258 3468 50  0000 L CNN
 F 1 "TestPoint" H 5258 3377 50  0000 L CNN
 F 2 "TestPoint:TestPoint_Pad_1.0x1.0mm" H 5400 3350 50  0001 C CNN
@@
 Connection ~ 5200 3350
 $Comp
-L Connector:TestPoint TPVAD3
+L Connector:TestPoint TPVAD1
 U 1 1 5EF29675
 P 5300 2850
-F 0 "TPVAD3" H 5358 2968 50  0000 L CNN
+F 0 "TPVAD1" H 5358 2968 50  0000 L CNN
 F 1 "TestPoint" H 5358 2877 50  0000 L CNN
 F 2 "TestPoint:TestPoint_Pad_1.0x1.0mm" H 5500 2850 50  0001 C CNN

Commit message: Placement première charge active 2nd try
Parts:
- renumbered TPVGS3 to TPVGS1
Changed lines of the file:
@@
 	5300 2850 8100 2850
 $Comp
-L Connector:TestPoint TPVGS3
+L Connector:TestPoint TPVGS1
 U 1 1 5EF29845
 P 7200 3900
-F 0 "TPVGS3" H 7258 4018 50  0000 L CNN
+F 0 "TPVGS1" H 7258 4018 50  0000 L CNN
 F 1 "TestPoint" H 7258 3927 50  0000 L CNN
 F 2 "TestPoint:TestPoint_Pad_1.0x1.0mm" H 7400 3900 50  0001 C CNN

Commit message: Defi releve!
Parts:
- removed J17: PowerMosSource, PCB:30ATerminal, symbol Connector:Screw_Terminal_01x01
Other:
- note added: "To a IXFN360N10T power mosfet\nSource connected to the 100W_ch-\n"
- note removed: "To a IXFN360N10T power mosfet\n"
Changed lines of the file:
@@
 VIN
-Wire Wire Line
-	8100 4100 8100 4350
 Wire Wire Line
 	5200 3800 5250 3800
@@
 	7450 3900 7450 4100
 $Comp
-L power:GNDA #PWR0206
-U 1 1 610FD9E1
-P 8100 4350
-F 0 "#PWR0206" H 8100 4100 50  0001 C CNN
-F 1 "GNDA" H 8105 4177 50  0000 C CNN
-F 2 "" H 8100 4350 50  0001 C CNN
-F 3 "" H 8100 4350 50  0001 C CNN
-	1    8100 4350
-	1    0    0    -1
-$EndComp
-$Comp
 L power:GNDA #PWR0204
 U 1 1 610FDDC3
@@
 	1    0    0    -1
 $EndComp
-$Comp
-L Connector:Screw_Terminal_01x01 J17
-U 1 1 61965D06
-P 8300 4100
-F 0 "J17" H 8380 4142 50  0000 L CNN
-F 1 "PowerMosSource" H 8380 4051 50  0000 L CNN
-F 2 "PCB:30ATerminal" H 8300 4100 50  0001 C CNN
-F 3 "~" H 8300 4100 50  0001 C CNN
-	1    8300 4100
-	1    0    0    -1
-$EndComp
 Text Notes 8750 4000 0    50   ~ 0
-To a IXFN360N10T power mosfet\n
-$Comp
-L Device:R R?
+To a IXFN360N10T power mosfet\nSource connected to the 100W_ch-\n
+$Comp
+L Device:R R?

Commit message: Petit ajustement pour accomoder le usb du arduino, pret pour routing
Parts:
- renumbered TPOA1 to OA1, TPOB1 to OB1, TPV+1 to V+3, TPV-1 to V-3, TPVAD1 to VAD3, TPVGS1 to VGS3
Changed lines of the file:
@@
 Connection ~ 4850 3750
 $Comp
-L Connector:TestPoint TPV-1
+L Connector:TestPoint V-3
 U 1 1 5EF281AD
 P 4100 4000
-F 0 "TPV-1" H 4158 4118 50  0000 L CNN
+F 0 "V-3" H 4158 4118 50  0000 L CNN
 F 1 "TestPoint" H 4158 4027 50  0000 L CNN
 F 2 "TestPoint:TestPoint_Pad_1.0x1.0mm" H 4300 4000 50  0001 C CNN
@@
 $EndComp
 $Comp
-L Connector:TestPoint TPV+1
+L Connector:TestPoint V+3
 U 1 1 5EF2916C
 P 5200 3350
-F 0 "TPV+1" H 5258 3468 50  0000 L CNN
+F 0 "V+3" H 5258 3468 50  0000 L CNN
 F 1 "TestPoint" H 5258 3377 50  0000 L CNN
 F 2 "TestPoint:TestPoint_Pad_1.0x1.0mm" H 5400 3350 50  0001 C CNN
@@
 Connection ~ 5200 3350
 $Comp
-L Connector:TestPoint TPVAD1
+L Connector:TestPoint VAD3
 U 1 1 5EF29675
 P 5300 2850
-F 0 "TPVAD1" H 5358 2968 50  0000 L CNN
+F 0 "VAD3" H 5358 2968 50  0000 L CNN
 F 1 "TestPoint" H 5358 2877 50  0000 L CNN
 F 2 "TestPoint:TestPoint_Pad_1.0x1.0mm" H 5500 2850 50  0001 C CNN
@@
 	5300 2850 8100 2850
 $Comp
-L Connector:TestPoint TPVGS1
+L Connector:TestPoint VGS3
 U 1 1 5EF29845
 P 7200 3900
-F 0 "TPVGS1" H 7258 4018 50  0000 L CNN
+F 0 "VGS3" H 7258 4018 50  0000 L CNN
 F 1 "TestPoint" H 7258 3927 50  0000 L CNN
 F 2 "TestPoint:TestPoint_Pad_1.0x1.0mm" H 7400 3900 50  0001 C CNN
@@
 $EndComp
 $Comp
-L Connector:TestPoint TPOA1
+L Connector:TestPoint OA1
 U 1 1 5EF2AA56
 P 5900 3900
-F 0 "TPOA1" H 5958 4018 50  0000 L CNN
+F 0 "OA1" H 5958 4018 50  0000 L CNN
 F 1 "TestPoint" H 5958 3927 50  0000 L CNN
 F 2 "TestPoint:TestPoint_Pad_1.0x1.0mm" H 6100 3900 50  0001 C CNN
@@
 $EndComp
 $Comp
-L Connector:TestPoint TPOB1
+L Connector:TestPoint OB1
 U 1 1 5EF2C651
 P 5900 4550
-F 0 "TPOB1" H 5958 4668 50  0000 L CNN
+F 0 "OB1" H 5958 4668 50  0000 L CNN
 F 1 "TestPoint" H 5958 4577 50  0000 L CNN
 F 2 "TestPoint:TestPoint_Pad_1.0x1.0mm" H 6100 4550 50  0001 C CNN

Commit message: retrait des test points inutiles
Parts:
- removed VAD3, VGS3: TestPoint, TestPoint:TestPoint_Pad_1.0x1.0mm, symbol Connector:TestPoint
Changed lines of the file:
@@
 	0    1    1    0
 $EndComp
-Wire Wire Line
-	4850 2850 5300 2850
 Connection ~ 4850 2850
 Wire Wire Line
@@
 Connection ~ 5200 3350
 $Comp
-L Connector:TestPoint VAD3
-U 1 1 5EF29675
-P 5300 2850
-F 0 "VAD3" H 5358 2968 50  0000 L CNN
-F 1 "TestPoint" H 5358 2877 50  0000 L CNN
-F 2 "TestPoint:TestPoint_Pad_1.0x1.0mm" H 5500 2850 50  0001 C CNN
-F 3 "~" H 5500 2850 50  0001 C CNN
-	1    5300 2850
-	1    0    0    -1
-$EndComp
-Connection ~ 5300 2850
-Wire Wire Line
-	5300 2850 8100 2850
-$Comp
-L Connector:TestPoint VGS3
-U 1 1 5EF29845
-P 7200 3900
-F 0 "VGS3" H 7258 4018 50  0000 L CNN
-F 1 "TestPoint" H 7258 3927 50  0000 L CNN
-F 2 "TestPoint:TestPoint_Pad_1.0x1.0mm" H 7400 3900 50  0001 C CNN
-F 3 "~" H 7400 3900 50  0001 C CNN
-	1    7200 3900
-	1    0    0    -1
-$EndComp
-$Comp
 L Connector:TestPoint OA1
 U 1 1 5EF2AA56
@@
 	1    0    0    -1
 $EndComp
-Wire Wire Line
-	7050 3900 7200 3900
-Connection ~ 7200 3900
-Wire Wire Line
-	7200 3900 7450 3900
 Wire Wire Line
 	5850 3900 5900 3900
@@
 	0    1    1    0
 $EndComp
+Wire Wire Line
+	7050 3900 7450 3900
+Wire Wire Line
+	4850 2850 8100 2850
 $EndSCHEMATC

Commit message: Debut routing cannaux passifs
Connections:
- net GND: no longer C101.1
- net GNDA: now also C101.1
Changed lines of the file:
@@
 Connection ~ 4100 4000
-$Comp
-L power:GND #PWR?
-U 1 1 5EDD7C87
-P 4100 4500
-AR Path="/5F349895/5EDD7C87" Ref="#PWR?"  Part="1"
-AR Path="/5F9E924D/5EDD7C87" Ref="#PWR?"  Part="1"
-AR Path="/5FA111F4/5EDD7C87" Ref="#PWR?"  Part="1"
-AR Path="/5FA373CA/5EDD7C87" Ref="#PWR?"  Part="1"
-AR Path="/5FA5E0C4/5EDD7C87" Ref="#PWR?"  Part="1"
-AR Path="/5FA85B69/5EDD7C87" Ref="#PWR?"  Part="1"
-AR Path="/5FAADC18/5EDD7C87" Ref="#PWR?"  Part="1"
-AR Path="/5FAD6864/5EDD7C87" Ref="#PWR?"  Part="1"
-AR Path="/5EF81810/5EDD7C87" Ref="#PWR?"  Part="1"
-AR Path="/5EFA1964/5EDD7C87" Ref="#PWR0199"  Part="1"
-F 0 "#PWR0199" H 4100 4250 50  0001 C CNN
-F 1 "GND" H 4105 4327 50  0000 C CNN
-F 2 "" H 4100 4500 50  0001 C CNN
-F 3 "" H 4100 4500 50  0001 C CNN
-	1    4100 4500
-	1    0    0    -1
-$EndComp
 $Comp
 L Device:C C?
@@
 Wire Wire Line
 	4850 2850 8100 2850
+$Comp
+L power:GNDA #PWR?
+U 1 1 5F0ACC3E
+P 4100 4500
+F 0 "#PWR?" H 4100 4250 50  0001 C CNN
+F 1 "GNDA" H 4105 4327 50  0000 C CNN
+F 2 "" H 4100 4500 50  0001 C CNN
+F 3 "" H 4100 4500 50  0001 C CNN
+	1    4100 4500
+	1    0    0    -1
+$EndComp
 $EndSCHEMATC
