File: VoltageIndiv.sch (KiCad schematic (older format))
At the start: 2 parts

Commit message: routing usb
Changed lines of the file:
@@
 $Descr A4 11693 8268
 encoding utf-8
-Sheet 6 80
+Sheet 9 80
 Title ""
 Date "2020-05-19"
@@
 AR Path="/5F37413F/5EC90889" Ref="R79"  Part="1"
 AR Path="/5F374143/5EC90889" Ref="R81"  Part="1"
-F 0 "R39" H 5770 4046 50  0000 L CNN
+F 0 "R45" H 5770 4046 50  0000 L CNN
 F 1 "100k" H 5770 3955 50  0000 L CNN
 F 2 "Resistor_SMD:R_0805_2012Metric" V 5630 4000 50  0001 C CNN
@@
 AR Path="/5F37413F/5EC91EB2" Ref="R78"  Part="1"
 AR Path="/5F374143/5EC91EB2" Ref="R80"  Part="1"
-F 0 "R38" H 5770 3546 50  0000 L CNN
+F 0 "R44" H 5770 3546 50  0000 L CNN
 F 1 "43k" H 5770 3455 50  0000 L CNN
 F 2 "Resistor_SMD:R_0805_2012Metric" V 5630 3500 50  0001 C CNN
@@
 AR Path="/5F37413F/60F963CD" Ref="#PWR0138"  Part="1"
 AR Path="/5F374143/60F963CD" Ref="#PWR0139"  Part="1"
-F 0 "#PWR053" H 5700 4050 50  0001 C CNN
+F 0 "#PWR056" H 5700 4050 50  0001 C CNN
 F 1 "GNDA" H 5705 4127 50  0000 C CNN
 F 2 "" H 5700 4300 50  0001 C CNN

Commit message: Debut routing cannaux passifs
Changed lines of the file:
@@
 $Descr A4 11693 8268
 encoding utf-8
-Sheet 9 80
+Sheet 39 80
 Title ""
 Date "2020-05-19"
@@
 AR Path="/5F37413F/5EC90889" Ref="R79"  Part="1"
 AR Path="/5F374143/5EC90889" Ref="R81"  Part="1"
-F 0 "R45" H 5770 4046 50  0000 L CNN
+F 0 "R75" H 5770 4046 50  0000 L CNN
 F 1 "100k" H 5770 3955 50  0000 L CNN
 F 2 "Resistor_SMD:R_0805_2012Metric" V 5630 4000 50  0001 C CNN
@@
 AR Path="/5F37413F/5EC91EB2" Ref="R78"  Part="1"
 AR Path="/5F374143/5EC91EB2" Ref="R80"  Part="1"
-F 0 "R44" H 5770 3546 50  0000 L CNN
+F 0 "R74" H 5770 3546 50  0000 L CNN
 F 1 "43k" H 5770 3455 50  0000 L CNN
 F 2 "Resistor_SMD:R_0805_2012Metric" V 5630 3500 50  0001 C CNN
@@
 AR Path="/5F37413F/60F963CD" Ref="#PWR0138"  Part="1"
 AR Path="/5F374143/60F963CD" Ref="#PWR0139"  Part="1"
-F 0 "#PWR056" H 5700 4050 50  0001 C CNN
+F 0 "#PWR0136" H 5700 4050 50  0001 C CNN
 F 1 "GNDA" H 5705 4127 50  0000 C CNN
 F 2 "" H 5700 4300 50  0001 C CNN
